Commit message: added depth camera front,back and sides

File: autonomous_data_sampling_ws/src/sim/rotors_simulator/rotors_description/urdf/rmf_obelix_moveit.xacro (robot description, xacro)
@@ -169,4 +169,24 @@
     <origin xyz="0 0 0.04" rpy="0 0 0" />
   </xacro:OS0-128>
+  <!-- Add a depth camera instead of lidar -->
+  <xacro:include filename="$(find realsense2_description)/urdf/_d455.urdf.xacro"/>
+  <xacro:sensor_d455 parent="${namespace}/base_link" name="${namespace}/camera" topics_ns="${namespace}/camera">
+    <origin xyz="0.04 0 0.04" rpy="0 0 0" />
+  </xacro:sensor_d455>
+    <!-- Add a depth camera instead of lidar -->
+  <xacro:include filename="$(find realsense2_description)/urdf/_d455.urdf.xacro"/>
+  <xacro:sensor_d455 parent="${namespace}/base_link" name="${namespace}/camera2" topics_ns="${namespace}/camera2">
+    <origin xyz="-0.04 0 0.04" rpy="0 0 -3.14" />
+  </xacro:sensor_d455>
+      <!-- Add a depth camera instead of lidar -->
+  <xacro:include filename="$(find realsense2_description)/urdf/_d455.urdf.xacro"/>
+  <xacro:sensor_d455 parent="${namespace}/base_link" name="${namespace}/camera3" topics_ns="${namespace}/camera3">
+    <origin xyz="0 0 0.04" rpy="0 0 -1.57" />
+  </xacro:sensor_d455>
+      <!-- Add a depth camera instead of lidar -->
+  <xacro:include filename="$(find realsense2_description)/urdf/_d455.urdf.xacro"/>
+  <xacro:sensor_d455 parent="${namespace}/base_link" name="${namespace}/camera4" topics_ns="${namespace}/camera4">
+    <origin xyz="-0.04 0 0.04" rpy="0 0 1.57" />
+  </xacro:sensor_d455>
   <!--Kinect-->
   <!-- position of kinect has to be changed in common_sensors/urdf/sensors/kinect_properties.urdf.xacro-->
