Commit message: Path planning from mesh and execution added

File: autonomous_data_sampling_ws/src/sim/realsense2_description/urdf/_d435.gazebo.xacro (robot description, xacro)
@@ -93,6 +93,6 @@
           <horizontal_fov>${85.2*deg_to_rad}</horizontal_fov>
           <image>
-            <width>128</width>
-            <height>72</height>
+            <width>64</width>
+            <height>48</height>
             <!--width>1280</width>
             <height>720</height-->

File: autonomous_data_sampling_ws/src/sim/rotors_simulator/rotors_description/urdf/rmf_obelix_base.xacro (robot description, xacro)
@@ -46,3 +46,8 @@
     <origin xyz="0 0 0.04" rpy="0 0 0" />
   </xacro:OS0-128>
+  <!-- Add an 0S0-128 lidar -->
+  <xacro:include filename="$(find lidar_description)/urdf/OS0-128.urdf.xacro"/>
+  <xacro:OS0-128 parent="${namespace}/base_link" name="/vegard/velodyne" topic="vegard_points" hz="10" lasers="32" samples="440" collision_range="0.3" min_range="0.3" max_range="50.0">
+    <origin xyz="0 0 0.04" rpy="0 0 0" />
+  </xacro:OS0-128>
 </robot>

File: autonomous_data_sampling_ws/src/sim/rotors_simulator/rotors_description/urdf/rmf_obelix_moveit.xacro (robot description, xacro)
@@ -170,23 +170,24 @@
   </xacro:OS0-128>
   <!-- Add a depth camera instead of lidar -->
-  <xacro:include filename="$(find realsense2_description)/urdf/_d455.urdf.xacro"/>
+  <!-- <xacro:include filename="$(find realsense2_description)/urdf/_d455.urdf.xacro"/>
   <xacro:sensor_d455 parent="${namespace}/base_link" name="${namespace}/camera" topics_ns="${namespace}/camera">
     <origin xyz="0.04 0 0.04" rpy="0 0 0" />
-  </xacro:sensor_d455>
+  </xacro:sensor_d455> -->
     <!-- Add a depth camera instead of lidar -->
-  <xacro:include filename="$(find realsense2_description)/urdf/_d455.urdf.xacro"/>
+  <!-- <xacro:include filename="$(find realsense2_description)/urdf/_d455.urdf.xacro"/>
   <xacro:sensor_d455 parent="${namespace}/base_link" name="${namespace}/camera2" topics_ns="${namespace}/camera2">
     <origin xyz="-0.04 0 0.04" rpy="0 0 -3.14" />
   </xacro:sensor_d455>
+   -->
       <!-- Add a depth camera instead of lidar -->
-  <xacro:include filename="$(find realsense2_description)/urdf/_d455.urdf.xacro"/>
+  <!-- <xacro:include filename="$(find realsense2_description)/urdf/_d455.urdf.xacro"/>
   <xacro:sensor_d455 parent="${namespace}/base_link" name="${namespace}/camera3" topics_ns="${namespace}/camera3">
     <origin xyz="0 0 0.04" rpy="0 0 -1.57" />
-  </xacro:sensor_d455>
+  </xacro:sensor_d455> -->
       <!-- Add a depth camera instead of lidar -->
-  <xacro:include filename="$(find realsense2_description)/urdf/_d455.urdf.xacro"/>
+  <!-- <xacro:include filename="$(find realsense2_description)/urdf/_d455.urdf.xacro"/>
   <xacro:sensor_d455 parent="${namespace}/base_link" name="${namespace}/camera4" topics_ns="${namespace}/camera4">
     <origin xyz="-0.04 0 0.04" rpy="0 0 1.57" />
-  </xacro:sensor_d455>
+  </xacro:sensor_d455> -->
   <!--Kinect-->
   <!-- position of kinect has to be changed in common_sensors/urdf/sensors/kinect_properties.urdf.xacro-->
